File: MUX_board/MUX_v2024_relay_board_32/MUX_v2024_relay_board_32.kicad_pcb (KiCad board)
At the start: 2 copper layers, 140 x 350 mm, 192 parts, among them K1 G5LE-1-VD, K10 G5LE-1-VD, K11 G5LE-1-VD, K12 G5LE-1-VD, K13 G5LE-1-VD, K14 G5LE-1-VD, K15 G5LE-1-VD, K16 G5LE-1-VD, K17 G5LE-1-VD, K18 G5LE-1-VD, K19 G5LE-1-VD, K2 G5LE-1-VD, K20 G5LE-1-VD, K21 G5LE-1-VD, K22 G5LE-1-VD, K23 G5LE-1-VD, K24 G5LE-1-VD, K25 G5LE-1-VD, K26 G5LE-1-VD, K27 G5LE-1-VD, K28 G5LE-1-VD, K29 G5LE-1-VD, K3 G5LE-1-VD, K30 G5LE-1-VD, K31 G5LE-1-VD, K32 G5LE-1-VD, K4 G5LE-1-VD, K5 G5LE-1-VD, K6 G5LE-1-VD, K7 G5LE-1-VD, K8 G5LE-1-VD, K9 G5LE-1-VD, Q1 STP16NF06L, Q10 STP16NF06L, Q11 STP16NF06L, Q12 STP16NF06L, Q13 STP16NF06L, Q14 STP16NF06L, Q15 STP16NF06L, Q16 STP16NF06L, Q17 STP16NF06L, Q18 STP16NF06L, Q19 STP16NF06L, Q2 STP16NF06L, Q20 STP16NF06L, Q21 STP16NF06L, Q22 STP16NF06L, Q23 STP16NF06L, Q24 STP16NF06L, Q25 STP16NF06L, Q26 STP16NF06L, Q27 STP16NF06L, Q28 STP16NF06L, Q29 STP16NF06L, Q3 STP16NF06L, Q30 STP16NF06L, Q31 STP16NF06L, Q32 STP16NF06L, Q4 STP16NF06L, Q5 STP16NF06L, Q6 STP16NF06L, Q7 STP16NF06L, Q8 STP16NF06L, Q9 STP16NF06L, U1 MCP23017_SP, U2 MCP23017_SP

Commit message: Updates MUX relay board
Routing:
- net Role x: track 408.4 -> 404.9 mm
- net Role y: track 408.4 -> 409.7 mm
- net Electrode 10: track 329.2 -> 328.0 mm
- net Role xx: track 357.1 -> 358.3 mm
- net Electrode 14: track 161.9 -> 160.8 mm
- net Electrode 12: track 243.1 -> 242.0 mm

Commit message: Fixes last errors on pcb
Parts:
- moved GND  PWR 6.83 mm to (40.0, 69.0)
Routing:
- net Electrode 8: track 427.3 -> 419.1 mm
- net 12V: track 1160.3 -> 1166.4 mm
- net Electrode 9: track 425.1 -> 428.1 mm
- net Electrode 11: track 336.5 -> 339.2 mm
- net Electrode 13: track 225.6 -> 228.1 mm
- net Electrode 15: track 127.4 -> 129.1 mm
- net Electrode 6: track 300.5 -> 301.1 mm
- net Electrode 3: track 213.1 -> 213.7 mm
- net Electrode 7: track 410.0 -> 410.5 mm
- net Role x: track 404.9 -> 404.3 mm
- net Electrode 2: track 148.8 -> 149.3 mm
- net Electrode 4: track 224.7 -> 225.3 mm
- net GND: vias 38 -> 42
Other:
- board text added: "MUX relays board 2/4 roles v2024 - OhmPi project"
- board text added: "UMONS GFA - 12-2022"

Commit message: Improves annotations on pcb board
Parts:
- Jumper 5V: renamed from Jumper 5V-12V
- Jumper E1: renamed from JP5
- Jumper E2: renamed from JP6
- Jumper E3: renamed from JP7
- Jumper E4: renamed from JP8
- Jumper E5: renamed from JP9
- Jumper E6: renamed from JP10
- Jumper E7: renamed from JP11
- Jumper E8: renamed from JP12
- moved REF** 2.00 mm to (35.4, 45.1)
- moved REF** 2.00 mm to (35.4, 385.1)
- moved REF** 2.00 mm to (35.4, 195.1)
- moved REF** 2.00 mm to (35.4, 85.1)
- moved REF** 2.00 mm to (35.4, 345.1)
- moved REF** 2.00 mm to (35.4, 235.1)
- moved REF** 1.00 mm to (166.4, 385.1)
- moved REF** 1.00 mm to (166.4, 235.1)
- moved REF** 1.00 mm to (166.4, 85.1)
- moved REF** 1.00 mm to (166.4, 345.1)
- moved REF** 1.00 mm to (166.4, 195.1)
- moved REF** 1.00 mm to (166.4, 45.1)
Other:
- board text added: "E1xx"
- board text added: "E1yy"
- board text added: "E2xx"
- board text added: "E2yy"
- board text added: "E3xx"
- board text added: "E3yy"
- board text added: "E4xx"
- board text added: "E4yy"
- board text added: "E5xx"
- board text added: "E5yy"
- board text added: "E6xx"
- board text added: "E6yy"
- board text added: "E7xx"
- board text added: "E7yy"
- board text added: "E8xx"
- board text added: "E8yy"
