File: MUX_board/2024.0.0/relay_board_32/MUX_v2024_relay_board_32.kicad_pcb (KiCad board)
At the start: 2 copper layers, 140 x 350 mm, 195 parts, among them K1 G5LE-1-VD, K10 G5LE-1-VD, K11 G5LE-1-VD, K12 G5LE-1-VD, K13 G5LE-1-VD, K14 G5LE-1-VD, K15 G5LE-1-VD, K16 G5LE-1-VD, K17 G5LE-1-VD, K18 G5LE-1-VD, K19 G5LE-1-VD, K2 G5LE-1-VD, K20 G5LE-1-VD, K21 G5LE-1-VD, K22 G5LE-1-VD, K23 G5LE-1-VD, K24 G5LE-1-VD, K25 G5LE-1-VD, K26 G5LE-1-VD, K27 G5LE-1-VD, K28 G5LE-1-VD, K29 G5LE-1-VD, K3 G5LE-1-VD, K30 G5LE-1-VD, K31 G5LE-1-VD, K32 G5LE-1-VD, K4 G5LE-1-VD, K5 G5LE-1-VD, K6 G5LE-1-VD, K7 G5LE-1-VD, K8 G5LE-1-VD, K9 G5LE-1-VD, Q1 STP16NF06L, Q10 STP16NF06L, Q11 STP16NF06L, Q12 STP16NF06L, Q13 STP16NF06L, Q14 STP16NF06L, Q15 STP16NF06L, Q16 STP16NF06L, Q17 STP16NF06L, Q18 STP16NF06L, Q19 STP16NF06L, Q2 STP16NF06L, Q20 STP16NF06L, Q21 STP16NF06L, Q22 STP16NF06L, Q23 STP16NF06L, Q24 STP16NF06L, Q25 STP16NF06L, Q26 STP16NF06L, Q27 STP16NF06L, Q28 STP16NF06L, Q29 STP16NF06L, Q3 STP16NF06L, Q30 STP16NF06L, Q31 STP16NF06L, Q32 STP16NF06L, Q4 STP16NF06L, Q5 STP16NF06L, Q6 STP16NF06L, Q7 STP16NF06L, Q8 STP16NF06L, Q9 STP16NF06L, U1 MCP23017_SP, U2 MCP23017_SP

Commit message: adds filtering capacitors on MCP23017
Parts:
- added C2: 100nF, Capacitor_THT:C_Disc_D7.0mm_W2.5mm_P5.00mm, F.Cu at (121.0, 376.8)
- added C3: 10uF, Capacitor_THT:CP_Radial_D6.3mm_P2.50mm, F.Cu at (120.4, 382.4)
- added C4: 10uF, Capacitor_THT:CP_Radial_D6.3mm_P2.50mm, F.Cu at (82.2, 382.4)
- C1: footprint Capacitor_THT:C_Disc_D8.0mm_W2.5mm_P5.00mm -> Capacitor_THT:C_Disc_D7.0mm_W2.5mm_P5.00mm
- moved R34 15.2 mm to (100.9, 357.8), turned to -90 degrees
- moved R33 15.1 mm to (106.0, 357.8), turned to -90 degrees
- moved C1 13.7 mm to (81.4, 376.8), turned to 0 degrees
- moved U2 6.56 mm to (45.0, 384.9)
- moved Addr2 3.56 mm to (112.1, 378.9)
- moved U1 2.94 mm to (157.7, 377.3)
- moved Addr1 2.56 mm to (107.7, 378.9)
- moved Electrodes IDC 1.56 mm to (94.3, 70.0)
- moved Jumper 5V 1.56 mm to (103.3, 348.4)
- moved Jumper x 1.56 mm to (148.5, 61.8)
- moved Jumper y 1.56 mm to (148.5, 44.8)
- moved K10 1.56 mm to (133.5, 309.9)
- moved K11 1.56 mm to (133.5, 273.0)
- moved K12 1.56 mm to (133.5, 236.0)
- moved K13 1.56 mm to (133.5, 199.1)
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Routing:
- net +5V: track 137.5 -> 152.6 mm
- net Addr2: track 52.0 -> 64.6 mm
- net Addr1: track 47.5 -> 57.7 mm
- net SD1: track 66.3 -> 62.2 mm
- net E9y: track 16.0 -> 18.6 mm
- net E10x: track 93.7 -> 95.5 mm
- net E9x: track 58.2 -> 59.8 mm
- net SCL1: track 68.3 -> 69.7 mm
- net E7y: track 91.1 -> 92.4 mm
- net E11x: track 129.3 -> 130.6 mm
- net E12x: track 164.8 -> 166.1 mm
- net E13x: track 200.3 -> 201.6 mm
- net E14x: track 235.8 -> 237.1 mm
- net E15x: track 271.3 -> 272.6 mm
- net E16x: track 306.8 -> 308.1 mm
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Other:
- board text added: "UMONS GFA - 05 - 2023"
- board text removed: "UMONS GFA - 12-2022"

Commit message: imrpoves labelling
Parts:
- moved Jumper y 1.00 mm to (148.5, 43.8)
Routing:
- net Role yy: track 377.0 -> 378.0 mm
Other:
- outline, holes or cut-outs redrawn
Changed lines of the file:
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@@
     (property "Sheetname" "")
     (attr through_hole)
-    (fp_text reference "Electrodes" (at 38.1 -6.26 180) (layer "F.SilkS")
-      (effects (font (size 1 1) (thickness 0.15)))
+    (fp_text reference "Electrodes" (at 38.1 -7.26 180) (layer "F.SilkS")
+      (effects (font (size 2 2) (thickness 0.3)))
     )
     (fp_text value "Screw_Terminal_01x16" (at 38.1 5.66 180) (layer "F.Fab")
@@
   )
   (footprint "Solder_jumper:Soder_jumper" (layer "F.Cu")
-    (at 148.470241 44.82)
+    (at 148.470241 43.82)
     (property "Sheetfile" "MUX_v2024_relay_board_32.kicad_sch")
     (property "Sheetname" "")
@@
     (property "Sheetname" "")
     (attr through_hole)
-    (fp_text reference "x  y  xx yy" (at 7.62 -6.26 180) (layer "F.SilkS")
-      (effects (font (size 1 1) (thickness 0.15)))
+    (fp_text reference "x  y  xx yy" (at 7.12 6.74 180) (layer "F.SilkS")
+      (effects (font (size 2 2) (thickness 0.3)))
     )
     (fp_text value "Screw_Terminal_01x04" (at 7.62 5.66 180) (layer "F.Fab")
@@
     (property "Sheetname" "")
     (attr through_hole)
-    (fp_text reference "GND  PWR" (at 2.54 -6.26 -90) (layer "F.SilkS")
-      (effects (font (size 1 1) (thickness 0.15)))
+    (fp_text reference "GND  PWR" (at 2.54 -7.26 -90) (layer "F.SilkS")
+      (effects (font (size 2 2) (thickness 0.15)))
     )
     (fp_text value "Relays Pwr" (at 2.54 5.66 -90) (layer "F.Fab")
@@
       (net 39 "Electrode 12") (pinfunction "B") (pintype "passive"))
   )
-  (gr_line (start 31 390) (end 31 40) (layer "Edge.Cuts") (width 0.1))
-  (gr_line (start 171 390) (end 171 40) (layer "Edge.Cuts") (width 0.1))
-  (gr_line (start 171 390) (end 31 390) (layer "Edge.Cuts") (width 0.1))
-  (gr_line (start 171 40) (end 31 40) (layer "Edge.Cuts") (width 0.1))
+  (gr_line (start 32.5 389.5) (end 31.5 388.5) (layer "Edge.Cuts") (width 0.1))
+  (gr_line (start 170.5 388.5) (end 171 387.5) (layer "Edge.Cuts") (width 0.1))
+  (gr_line (start 170.5 41.5) (end 169.5 40.5) (layer "Edge.Cuts") (width 0.1))
+  (gr_line (start 31 387.5) (end 31 42.5) (layer "Edge.Cuts") (width 0.1))
+  (gr_line (start 169.5 40.5) (end 168.5 40) (layer "Edge.Cuts") (width 0.1))
+  (gr_line (start 33.5 390) (end 32.5 389.5) (layer "Edge.Cuts") (width 0.1))
+  (gr_line (start 171 387.5) (end 171 42.5) (layer "Edge.Cuts") (width 0.1))
+  (gr_line (start 31.5 388.5) (end 31 387.5) (layer "Edge.Cuts") (width 0.1))
+  (gr_line (start 168.5 390) (end 33.5 390) (layer "Edge.Cuts") (width 0.1))
+  (gr_line (start 169.5 389.5) (end 170.5 388.5) (layer "Edge.Cuts") (width 0.1))
+  (gr_line (start 32.5 40.5) (end 31.5 41.5) (layer "Edge.Cuts") (width 0.1))
+  (gr_line (start 31.5 41.5) (end 31 42.5) (layer "Edge.Cuts") (width 0.1))
+  (gr_line (start 168.5 40) (end 33.5 40) (layer "Edge.Cuts") (width 0.1))
+  (gr_line (start 171 42.5) (end 170.5 41.5) (layer "Edge.Cuts") (width 0.1))
+  (gr_line (start 33.5 40) (end 32.5 40.5) (layer "Edge.Cuts") (width 0.1))
+  (gr_line (start 168.5 390) (end 169.5 389.5) (layer "Edge.Cuts") (width 0.1))
   (gr_text "E1yy" (at 110.063813 106.735453) (layer "F.SilkS")
     (effects (font (size 1.5 1.5) (thickness 0.1)))
@@
     (effects (font (size 1.8 1.8) (thickness 0.3)))
   )
-  (gr_text "MUX relays board 2/4 roles v2024 - OhmPi project" (at 32.335241 358.4 90) (layer "F.SilkS")
+  (gr_text "MUX relays board 2/4 roles v2024 - OhmPi project" (at 33.335241 310.4 90) (layer "F.SilkS")
     (effects (font (size 1.5 1.5) (thickness 0.3)))
   )
@@
     (effects (font (size 2.5 2.5) (thickness 0.3)))
   )
-  (gr_text "UMONS GFA - 05 - 2023" (at 154.135241 388.9) (layer "F.SilkS")
+  (gr_text "UMONS GFA - 05 - 2023" (at 148.635241 388.9) (layer "F.SilkS")
     (effects (font (size 1.5 1.5) (thickness 0.3)))
   )
@@
   (segment (start 138.469263 250.034022) (end 138.469263 213.034022) (width 2) (layer "F.Cu") (net 61))
   (segment (start 138.469263 213.034022) (end 138.469263 174.965978) (width 2) (layer "F.Cu") (net 61))
+  (segment (start 149.970241 44.02) (end 149.970241 45.02) (width 2) (layer "F.Cu") (net 61))
   (segment (start 156.070241 53.3) (end 156.070241 51.12) (width 2) (layer "F.Cu") (net 61))
   (segment (start 133.420241 328.360777) (end 134.074464 328.360777) (width 2) (layer "F.Cu") (net 61))
